Commit message: added visualisation in Rviz

File: urdf/project_1_group_2.urdf.xacro (robot description, xacro)
@@ -35,19 +35,29 @@
       </visual>
   </xacro:macro>
+<!--
+  # Add this before base link
+<link name="dummy_link"></link>
+# Add this after base link
+<joint name="dummy_joint" type="fixed">
+    <origin rpy="0 0 0" xyz="0 0 0" />
+    <parent link="dummy_link"/>
+    <child link="base_link"/>
+</joint>
+   -->
   <link
     name="base_link">
     <inertial>
       <origin
-        xyz="0.219542185844718 -0.489097435985613 0.253171163731009"
-        rpy="0 0 0" />
-      <mass
-        value="45.0255547584039" />
-      <inertia
-        ixx="3.47370213259269"
-        ixy="8.68638754770634E-06"
-        ixz="1.28817771727052E-06"
-        iyy="1.51493007257673"
-        iyz="0.0559660105211115"
-        izz="4.32787408102168" />
+        xyz="0.219542184923656 0.253147662670064 0.488981343790689"
+        rpy="0 0 0" />
+      <mass
+        value="1" />
+      <inertia
+        ixx="3.47686976214323"
+        ixy="1.28363813560472E-06"
+        ixz="-8.67881754875189E-06"
+        iyy="4.33091580677011"
+        iyz="-0.0565812633669083"
+        izz="1.5150564663539" />
     </inertial>
     <visual>
@@ -79,15 +89,15 @@
     <inertial>
       <origin
-        xyz="2.86075080291326E-08 0.0749063419355981 0.00254051949689649"
-        rpy="0 0 0" />
-      <mass
-        value="0.295424107267104" />
-      <inertia
-        ixx="0.000710809060839364"
-        ixy="1.53957020749097E-10"
-        ixz="3.53322320504462E-10"
+        xyz="2.86075080291326E-08 -0.0749063419355981 -0.00254051949689645"
+        rpy="0 0 0" />
+      <mass
+        value="5.295424107267105" />
+      <inertia
+        ixx="0.000710809060839366"
+        ixy="-1.53957020615015E-10"
+        ixz="-3.53322320543782E-10"
         iyy="0.000104054571155282"
-        iyz="3.85934455800396E-05"
-        izz="0.000690101015602261" />
+        iyz="3.85934455800395E-05"
+        izz="0.000690101015602262" />
     </inertial>
     <visual>
@@ -117,8 +127,8 @@
   <joint
     name="steering_joint_1"
-    type="continuous">
-    <origin
-      xyz="0.0709516994137151 -0.734196139704711 0.0381336482199598"
-      rpy="1.5707963267949 0 -1.64845028267497" />
+    type="revolute">
+    <origin
+      xyz="0.070952 -0.7342 0.035594"
+      rpy="-1.5708 0 -1.5708" />
     <parent
       link="base_link" />
@@ -127,4 +137,9 @@
     <axis
       xyz="0 1 0" />
+    <limit
+      lower="-3.14"
+      upper="3.14"
+      effort="10"
+      velocity="10" />
   </joint>
   <link
@@ -132,14 +147,14 @@
     <inertial>
       <origin
-        xyz="-1.11022302462516E-16 0.0328469418204771 -1.11022302462516E-16"
+        xyz="0 0.0251005990323743 0"
         rpy="0 0 0" />
       <mass
         value="0.217134053712094" />
       <inertia
-        ixx="0.000126052696684197"
-        ixy="-6.05628557286825E-20"
-        ixz="-1.01643953670516E-20"
+        ixx="0.000126052696684198"
+        ixy="-3.30911918449584E-21"
+        ixz="6.7762635780344E-21"
         iyy="0.000159854355976214"
-        iyz="-1.22819777351874E-19"
+        iyz="-7.03947290074457E-21"
         izz="0.000126052696684198" />
     </inertial>
@@ -172,6 +187,6 @@
     type="continuous">
     <origin
-      xyz="0 0.0234950000000013 0.0304806572118972"
-      rpy="1.5707963267949 0 1.16336545532605" />
+      xyz="0 -0.0234950000000001 -0.040767"
+      rpy="-1.5707963267949 0 -1.16226628629428" />
     <parent
       link="steering_wheel_1" />
@@ -185,5 +200,5 @@
     <inertial>
       <origin
-        xyz="-2.77555756156289E-16 0.033142685248773 -6.93671252038897E-06"
+        xyz="0 0.0380963424606702 -6.9367125220543E-06"
         rpy="0 0 0" />
       <mass
@@ -191,115 +206,120 @@
       <inertia
         ixx="0.00664149361787531"
-        ixy="-5.32614317233504E-18"
+        ixy="3.02337822610582E-19"
+        ixz="2.16840434497101E-19"
+        iyy="0.0114725337233255"
+        iyz="5.01717636400841E-07"
+        izz="0.00664244711710664" />
+    </inertial>
+    <visual>
+      <origin
+        xyz="0 0 0"
+        rpy="0 0 0" />
+      <geometry>
+        <mesh
+          filename="package://project_1_group_2/meshes/tire_1.STL" />
+      </geometry>
+      <material
+        name="">
+        <color
+          rgba="0.6 0.6 0.6 1" />
+      </material>
+    </visual>
+    <collision>
+      <origin
+        xyz="0 0 0"
+        rpy="0 0 0" />
+      <geometry>
+        <mesh
+          filename="package://project_1_group_2/meshes/tire_1.STL" />
+      </geometry>
+    </collision>
+  </link>
+  <joint
+    name="tire_1_joint"
+    type="fixed">
+    <origin
+      xyz="0 -0.0127000000000001 0"
+      rpy="0 0 0" />
+    <parent
+      link="wheel_1" />
+    <child
+      link="tire_1" />
+    <axis
+      xyz="0 0 0" />
+  </joint>
+  <link
+    name="steering_wheel_2">
+    <inertial>
+      <origin
+        xyz="2.86075079181103E-08 0.074906341935598 0.00254051949689649"
+        rpy="0 0 0" />
+      <mass
+        value="5.295424107267105" />
+      <inertia
+        ixx="0.000710809060839365"
+        ixy="1.53957021878157E-10"
+        ixz="3.53322320610221E-10"
+        iyy="0.000104054571155282"
+        iyz="3.85934455800397E-05"
+        izz="0.000690101015602261" />
+    </inertial>
+    <visual>
+      <origin
+        xyz="0 0 0"
+        rpy="0 0 0" />
+      <geometry>
+        <mesh
+          filename="package://project_1_group_2/meshes/steering_wheel_2.STL" />
+      </geometry>
+      <material
+        name="">
+        <color
+          rgba="1 0.168627450980392 0.168627450980392 1" />
+      </material>
+    </visual>
+    <collision>
+      <origin
+        xyz="0 0 0"
+        rpy="0 0 0" />
+      <geometry>
+        <mesh
+          filename="package://project_1_group_2/meshes/steering_wheel_2.STL" />
+      </geometry>
+    </collision>
+  </link>
+  <joint
+    name="steering_joint_2"
+    type="revolute">
+    <origin
+      xyz="0.36813 -0.7342 0.035594"
+      rpy="1.5708 0 1.5708" />
+    <parent
+      link="base_link" />
+    <child
+      link="steering_wheel_2" />
+    <axis
+      xyz="0 1 0" />
+    <limit
+      lower="-3.14"
+      upper="3.14"
+      effort="100"
+      velocity="10" />
+  </joint>
+  <link
+    name="wheel_2">
+    <inertial>
+      <origin
+        xyz="0 0.0251005990323743 0"
+        rpy="0 0 0" />
+      <mass
+        value="0.217134053712094" />
+      <inertia
+        ixx="0.000126052696684198"
+        ixy="-2.42959470068895E-21"
         ixz="0"
-        iyy="0.0114725337233255"
-        iyz="5.01717636383831E-07"
-        izz="0.00664244711710664" />
-    </inertial>
-    <visual>
-      <origin
-        xyz="0 0 0"
-        rpy="0 0 0" />
-      <geometry>
-        <mesh
-          filename="package://project_1_group_2/meshes/tire_1.STL" />
-      </geometry>
-      <material
-        name="">
-        <color
-          rgba="0.6 0.6 0.6 1" />
-      </material>
-    </visual>
-    <collision>
-      <origin
-        xyz="0 0 0"
-        rpy="0 0 0" />
-      <geometry>
-        <mesh
-          filename="package://project_1_group_2/meshes/tire_1.STL" />
-      </geometry>
-    </collision>
-  </link>
-  <joint
-    name="tire_joint_1"
-    type="fixed">
-    <origin
-      xyz="0 0 0"
-      rpy="0 0 0" />
-    <parent
-      link="wheel_1" />
-    <child
-      link="tire_1" />
-    <axis
-      xyz="0 0 0" />
-  </joint>
-  <link
-    name="steering_wheel_2">
-    <inertial>
-      <origin
-        xyz="2.86075079181103E-08 0.0749063419355979 0.0025405194968966"
-        rpy="0 0 0" />
-      <mass
-        value="0.295424107267104" />
-      <inertia
-        ixx="0.000710809060839366"
-        ixy="1.53957022007787E-10"
-        ixz="3.53322320524791E-10"
-        iyy="0.000104054571155282"
-        iyz="3.85934455800392E-05"
-        izz="0.000690101015602263" />
-    </inertial>
-    <visual>
-      <origin
-        xyz="0 0 0"
-        rpy="0 0 0" />
-      <geometry>
-        <mesh
-          filename="package://project_1_group_2/meshes/steering_wheel_2.STL" />
-      </geometry>
-      <material
-        name="">
-        <color
-          rgba="1 0.168627450980392 0.168627450980392 1" />
-      </material>
-    </visual>
-    <collision>
-      <origin
-        xyz="0 0 0"
-        rpy="0 0 0" />
-      <geometry>
-        <mesh
-          filename="package://project_1_group_2/meshes/steering_wheel_2.STL" />
-      </geometry>
-    </collision>
-  </link>
-  <joint
-    name="steering_joint_2"
-    type="continuous">
-    <origin
-      xyz="0.368131699413715 -0.734196139704711 0.0381336482199601"
-      rpy="1.5707963267949 0 1.46985194767708" />
-    <parent
-      link="base_link" />
-    <child
-      link="steering_wheel_2" />
-    <axis
-      xyz="0 1 0" />
-  </joint>
-  <link
-    name="wheel_2">
-    <inertial>
-      <origin
-        xyz="-1.11022302462516E-16 0.0327404142384009 4.85722573273506E-17"
-        rpy="0 0 0" />
-      <mass
-        value="0.217134053712094" />
-      <inertia
-        ixx="0.000126052696684197"
-        ixy="-1.40607469244214E-19"
-        ixz="4.58162463473438E-22"
         iyy="0.000159854355976214"
-        iyz="4.6915870035985E-20"
-        izz="0.000126052696684197" />
+        iyz="-1.47427383956479E-20"
+        izz="0.000126052696684198" />
     </inertial>
     <visual>
@@ -331,6 +351,6 @@
     type="continuous">
     <origin
-      xyz="0 0.023495 0.030587184793973"
-      rpy="1.5707963267949 0 0" />
+      xyz="0 0.0234950000000022 0.0407670000000003"
+      rpy="1.5707963267949 0 0.927408187420047" />
     <parent
       link="steering_wheel_2" />
@@ -344,5 +364,5 @@
     <inertial>
       <origin
-        xyz="-5.55111512312578E-16 0.0330361576666969 -6.93671252204042E-06"
+        xyz="-5.55111512312578E-17 0.0380963424606702 -6.93671252216532E-06"
         rpy="0 0 0" />
       <mass
@@ -350,8 +370,8 @@
       <inertia
         ixx="0.00664149361787532"
-        ixy="-2.23887748618257E-17"
-        ixz="-2.02295290606123E-20"
+        ixy="5.1086674631275E-20"
+        ixz="-2.16840434497101E-19"
         iyy="0.0114725337233255"
-        iyz="5.01717636407576E-07"
+        iyz="5.01717636401181E-07"
         izz="0.00664244711710664" />
     </inertial>
@@ -384,5 +404,5 @@
     type="fixed">
     <origin
-      xyz="0 0 0"
+      xyz="0 -0.0126999999999999 0"
       rpy="0 0 0" />
     <parent
@@ -397,5 +417,5 @@
     <inertial>
       <origin
-        xyz="0 -0.00394110038134092 0"
+        xyz="0 -0.00140110038134092 0"
         rpy="0 0 0" />
       <mass
@@ -403,8 +423,8 @@
       <inertia
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